Commit message: Renamed dae directory to lexus_model

File: config/urdf/lexus_model.urdf (robot description, URDF)
Before this commit: robot lexus, 2 links, 1 joints
Links:
- link lexus_model: geometry visual mesh filename=package://autoware_mini/config/urdf/lexus_model/Exterior.dae scale=1.0 1.02346 1.041

File: config/urdf/lexus_shadow.urdf (robot description, URDF)
Before this commit: robot lexus_shadow, 1 links, 0 joints
Links:
- link lexus_shadow: geometry visual mesh filename=package://autoware_mini/config/urdf/lexus_model/Exterior.dae scale=1.0 1.02346 1.041

Commit message: Updated lexus baselink to 0,0,0

File: config/urdf/lexus_model.urdf (robot description, URDF)
Before this commit: robot lexus, 2 links, 1 joints
Links:
- link lexus_model: geometry visual mesh filename=package://autoware_mini/config/urdf/lexus_model/Exterior.dae scale=1.0 1.0 1.0

File: config/urdf/lexus_shadow.urdf (robot description, URDF)
Before this commit: robot lexus_shadow, 1 links, 0 joints
Links:
- link lexus_shadow: geometry visual mesh filename=package://autoware_mini/config/urdf/lexus_model/Exterior.dae scale=1.0 1.0 1.0
